File: LastAcolyte6.kicad_pcb (KiCad board)
At the start: 4 copper layers, 100 x 100 mm, 85 parts, among them J1 Conn_02x23_Odd_Even, J10 DualPower_USB_B, J11 Conn_01x06, J2 DE9_Plug, J3 Conn_02x05_Odd_Even, J4 DE9_Plug, J5 DE15_Receptacle_HighDensity, J6 AudioJack3, J7 Mini-DIN-6, J8 Mini-DIN-6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

Commit message: Add files via upload
Connections:
- J1 pad 1: PHI2 -> ~{ZERO}
- J1 pad 10: /B4 -> /A4
- J1 pad 12: /B3 -> /A3
- J1 pad 14: /A18 -> /A2
- J1 pad 16: /A17 -> /A1
- J1 pad 18: /A16 -> /A0
- J1 pad 22: /A7 -> /B7
- J1 pad 24: /A6 -> /B6
- J1 pad 26: /A5 -> /B5
- J1 pad 28: /A4 -> /B4
- J1 pad 3: ~{ZERO} -> /A18
- J1 pad 30: /A3 -> /B3
- J1 pad 32: /A2 -> RDY
- J1 pad 34: /A1 -> ~{RD}
- J1 pad 36: /A0 -> ~{WR}
- J1 pad 4: /B7 -> /A7
- J1 pad 40: RDY -> PHI2
- J1 pad 5: ~{RD} -> /A17
- J1 pad 6: /B6 -> /A6
- J1 pad 7: ~{WR} -> /A16
- J1 pad 8: /B5 -> /A5
Changed lines of the file:
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@@
       (stroke (width 0.1) (type solid)) (layer "F.Fab"))
     (pad "1" thru_hole rect (at 0 0) (size 1.7 1.7) (drill 1) (layers "*.Cu" "*.Mask")
-      (net 132 "PHI2") (pinfunction "Pin_1") (pintype "passive"))
+      (net 167 "~{ZERO}") (pinfunction "Pin_1") (pintype "passive"))
     (pad "2" thru_hole oval (at 2.54 0) (size 1.7 1.7) (drill 1) (layers "*.Cu" "*.Mask")
       (net 1 "+5V") (pinfunction "Pin_2") (pintype "passive"))
     (pad "3" thru_hole oval (at 0 2.54) (size 1.7 1.7) (drill 1) (layers "*.Cu" "*.Mask")
-      (net 167 "~{ZERO}") (pinfunction "Pin_3") (pintype "passive"))
+      (net 111 "/A18") (pinfunction "Pin_3") (pintype "passive"))
     (pad "4" thru_hole oval (at 2.54 2.54) (size 1.7 1.7) (drill 1) (layers "*.Cu" "*.Mask")
-      (net 88 "/B7") (pinfunction "Pin_4") (pintype "passive"))
+      (net 82 "/A7") (pinfunction "Pin_4") (pintype "passive"))
     (pad "5" thru_hole oval (at 0 5.08) (size 1.7 1.7) (drill 1) (layers "*.Cu" "*.Mask")
-      (net 91 "~{RD}") (pinfunction "Pin_5") (pintype "passive"))
+      (net 94 "/A17") (pinfunction "Pin_5") (pintype "passive"))
     (pad "6" thru_hole oval (at 2.54 5.08) (size 1.7 1.7) (drill 1) (layers "*.Cu" "*.Mask")
-      (net 87 "/B6") (pinfunction "Pin_6") (pintype "passive"))
+      (net 81 "/A6") (pinfunction "Pin_6") (pintype "passive"))
     (pad "7" thru_hole oval (at 0 7.62) (size 1.7 1.7) (drill 1) (layers "*.Cu" "*.Mask")
-      (net 92 "~{WR}") (pinfunction "Pin_7") (pintype "passive"))
+      (net 95 "/A16") (pinfunction "Pin_7") (pintype "passive"))
     (pad "8" thru_hole oval (at 2.54 7.62) (size 1.7 1.7) (drill 1) (layers "*.Cu" "*.Mask")
-      (net 86 "/B5") (pinfunction "Pin_8") (pintype "passive"))
+      (net 80 "/A5") (pinfunction "Pin_8") (pintype "passive"))
     (pad "9" thru_hole oval (at 0 10.16) (size 1.7 1.7) (drill 1) (layers "*.Cu" "*.Mask")
       (net 2 "GND") (pinfunction "Pin_9") (pintype "passive"))
     (pad "10" thru_hole oval (at 2.54 10.16) (size 1.7 1.7) (drill 1) (layers "*.Cu" "*.Mask")
-      (net 85 "/B4") (pinfunction "Pin_10") (pintype "passive"))
+      (net 79 "/A4") (pinfunction "Pin_10") (pintype "passive"))
     (pad "11" thru_hole oval (at 0 12.7) (size 1.7 1.7) (drill 1) (layers "*.Cu" "*.Mask")
       (net 112 "/A15") (pinfunction "Pin_11") (pintype "passive"))
     (pad "12" thru_hole oval (at 2.54 12.7) (size 1.7 1.7) (drill 1) (layers "*.Cu" "*.Mask")
-      (net 84 "/B3") (pinfunction "Pin_12") (pintype "passive"))
+      (net 78 "/A3") (pinfunction "Pin_12") (pintype "passive"))
     (pad "13" thru_hole oval (at 0 15.24) (size 1.7 1.7) (drill 1) (layers "*.Cu" "*.Mask")
       (net 96 "/A14") (pinfunction "Pin_13") (pintype "passive"))
     (pad "14" thru_hole oval (at 2.54 15.24) (size 1.7 1.7) (drill 1) (layers "*.Cu" "*.Mask")
-      (net 111 "/A18") (pinfunction "Pin_14") (pintype "passive"))
+      (net 77 "/A2") (pinfunction "Pin_14") (pintype "passive"))
     (pad "15" thru_hole oval (at 0 17.78) (size 1.7 1.7) (drill 1) (layers "*.Cu" "*.Mask")
       (net 110 "/A13") (pinfunction "Pin_15") (pintype "passive"))
     (pad "16" thru_hole oval (at 2.54 17.78) (size 1.7 1.7) (drill 1) (layers "*.Cu" "*.Mask")
-      (net 94 "/A17") (pinfunction "Pin_16") (pintype "passive"))
+      (net 76 "/A1") (pinfunction "Pin_16") (pintype "passive"))
     (pad "17" thru_hole oval (at 0 20.32) (size 1.7 1.7) (drill 1) (layers "*.Cu" "*.Mask")
       (net 97 "/A12") (pinfunction "Pin_17") (pintype "passive"))
     (pad "18" thru_hole oval (at 2.54 20.32) (size 1.7 1.7) (drill 1) (layers "*.Cu" "*.Mask")
-      (net 95 "/A16") (pinfunction "Pin_18") (pintype "passive"))
+      (net 75 "/A0") (pinfunction "Pin_18") (pintype "passive"))
     (pad "19" thru_hole oval (at 0 22.86) (size 1.7 1.7) (drill 1) (layers "*.Cu" "*.Mask")
       (net 107 "/A11") (pinfunction "Pin_19") (pintype "passive"))
@@
       (net 106 "/A10") (pinfunction "Pin_21") (pintype "passive"))
     (pad "22" thru_hole oval (at 2.54 25.4) (size 1.7 1.7) (drill 1) (layers "*.Cu" "*.Mask")
-      (net 82 "/A7") (pinfunction "Pin_22") (pintype "passive"))
+      (net 88 "/B7") (pinfunction "Pin_22") (pintype "passive"))
     (pad "23" thru_hole oval (at 0 27.94) (size 1.7 1.7) (drill 1) (layers "*.Cu" "*.Mask")
       (net 108 "/A9") (pinfunction "Pin_23") (pintype "passive"))
     (pad "24" thru_hole oval (at 2.54 27.94) (size 1.7 1.7) (drill 1) (layers "*.Cu" "*.Mask")
-      (net 81 "/A6") (pinfunction "Pin_24") (pintype "passive"))
+      (net 87 "/B6") (pinfunction "Pin_24") (pintype "passive"))
     (pad "25" thru_hole oval (at 0 30.48) (size 1.7 1.7) (drill 1) (layers "*.Cu" "*.Mask")
       (net 109 "/A8") (pinfunction "Pin_25") (pintype "passive"))
     (pad "26" thru_hole oval (at 2.54 30.48) (size 1.7 1.7) (drill 1) (layers "*.Cu" "*.Mask")
-      (net 80 "/A5") (pinfunction "Pin_26") (pintype "passive"))
+      (net 86 "/B5") (pinfunction "Pin_26") (pintype "passive"))
     (pad "27" thru_hole oval (at 0 33.02) (size 1.7 1.7) (drill 1) (layers "*.Cu" "*.Mask")
       (net 2 "GND") (pinfunction "Pin_27") (pintype "passive"))
     (pad "28" thru_hole oval (at 2.54 33.02) (size 1.7 1.7) (drill 1) (layers "*.Cu" "*.Mask")
-      (net 79 "/A4") (pinfunction "Pin_28") (pintype "passive"))
+      (net 85 "/B4") (pinfunction "Pin_28") (pintype "passive"))
     (pad "29" thru_hole oval (at 0 35.56) (size 1.7 1.7) (drill 1) (layers "*.Cu" "*.Mask")
       (net 98 "/D0") (pinfunction "Pin_29") (pintype "passive"))
     (pad "30" thru_hole oval (at 2.54 35.56) (size 1.7 1.7) (drill 1) (layers "*.Cu" "*.Mask")
-      (net 78 "/A3") (pinfunction "Pin_30") (pintype "passive"))
+      (net 84 "/B3") (pinfunction "Pin_30") (pintype "passive"))
     (pad "31" thru_hole oval (at 0 38.1) (size 1.7 1.7) (drill 1) (layers "*.Cu" "*.Mask")
       (net 99 "/D1") (pinfunction "Pin_31") (pintype "passive"))
     (pad "32" thru_hole oval (at 2.54 38.1) (size 1.7 1.7) (drill 1) (layers "*.Cu" "*.Mask")
-      (net 77 "/A2") (pinfunction "Pin_32") (pintype "passive"))
+      (net 153 "RDY") (pinfunction "Pin_32") (pintype "passive"))
     (pad "33" thru_hole oval (at 0 40.64) (size 1.7 1.7) (drill 1) (layers "*.Cu" "*.Mask")
       (net 100 "/D2") (pinfunction "Pin_33") (pintype "passive"))
     (pad "34" thru_hole oval (at 2.54 40.64) (size 1.7 1.7) (drill 1) (layers "*.Cu" "*.Mask")
-      (net 76 "/A1") (pinfunction "Pin_34") (pintype "passive"))
+      (net 91 "~{RD}") (pinfunction "Pin_34") (pintype "passive"))
     (pad "35" thru_hole oval (at 0 43.18) (size 1.7 1.7) (drill 1) (layers "*.Cu" "*.Mask")
       (net 101 "/D3") (pinfunction "Pin_35") (pintype "passive"))
     (pad "36" thru_hole oval (at 2.54 43.18) (size 1.7 1.7) (drill 1) (layers "*.Cu" "*.Mask")
-      (net 75 "/A0") (pinfunction "Pin_36") (pintype "passive"))
+      (net 92 "~{WR}") (pinfunction "Pin_36") (pintype "passive"))
     (pad "37" thru_hole oval (at 0 45.72) (size 1.7 1.7) (drill 1) (layers "*.Cu" "*.Mask")
       (net 102 "/D4") (pinfunction "Pin_37") (pintype "passive"))
@@
       (net 103 "/D5") (pinfunction "Pin_39") (pintype "passive"))
     (pad "40" thru_hole oval (at 2.54 48.26) (size 1.7 1.7) (drill 1) (layers "*.Cu" "*.Mask")
-      (net 153 "RDY") (pinfunction "Pin_40") (pintype "passive"))
+      (net 132 "PHI2") (pinfunction "Pin_40") (pintype "passive"))
     (pad "41" thru_hole oval (at 0 50.8) (size 1.7 1.7) (drill 1) (layers "*.Cu" "*.Mask")
       (net 104 "/D6") (pinfunction "Pin_41") (pintype "passive"))

Commit message: Add files via upload
Parts:
- added C11: C_Small, Capacitor_THT:C_Disc_D3.0mm_W2.0mm_P2.50mm, F.Cu at (95.2, 108.9)
- added C12: C_Small, Capacitor_THT:C_Disc_D3.0mm_W2.0mm_P2.50mm, F.Cu at (82.6, 134.6)
- added C29: C_Small, Capacitor_THT:C_Disc_D3.0mm_W2.0mm_P2.50mm, F.Cu at (92.7, 134.6)
- added R5: R_US, Resistor_THT:R_Axial_DIN0207_L6.3mm_D2.5mm_P2.54mm_Vertical, F.Cu at (102.2, 76.2)
- added U11: 74AHCT245, LastAcolyte6:SOIC-20-Adj_7.5x12.8mm_P1.27mm, F.Cu at (87.0, 107.3)
- added U13: 74AHCT1G125, Package_TO_SOT_SMD:SOT-23-5_HandSoldering, F.Cu at (101.6, 139.1)
- added U8: 74HCT166, Package_SO:SOIC-16_3.9x9.9mm_P1.27mm, F.Cu at (82.6, 141.6)
- added U9: 74HCT166, Package_SO:SOIC-16_3.9x9.9mm_P1.27mm, F.Cu at (92.7, 141.6)
- U14: value TXB0104D -> 74AHCT1G125; footprint Package_SO:SOIC-14_3.9x8.7mm_P1.27mm -> Package_TO_SOT_SMD:SOT-23-5_HandSoldering
- moved R4 60.5 mm to (154.9, 84.5), turned to -90 degrees
- moved C27 54.5 mm to (102.9, 134.6), turned to 180 degrees
- moved C9 42.0 mm to (80.0, 85.1), turned to -90 degrees
- moved RN2 35.8 mm to (80.0, 148.6)
- moved U16 31.1 mm to (129.5, 149.2), turned to -90 degrees
- moved C21 30.2 mm to (122.6, 94.2)
- moved C5 30.2 mm to (104.8, 89.1)
- moved C13 30.2 mm to (117.5, 85.9)
- moved U1 30.2 mm to (113.7, 94.8)
- moved X1 28.7 mm to (118.8, 127.0)
- moved C4 28.7 mm to (113.7, 131.4)
- moved C25 26.8 mm to (154.9, 150.8), turned to -90 degrees
- moved C26 26.2 mm to (137.8, 150.8), turned to -90 degrees
- moved G1000 26.2 mm to (109.2, 106.7), turned to 0 degrees
- moved C18 24.4 mm to (129.5, 140.3)
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Connections:
- C27 pad 2: +3.3V -> +5V
- J11 pad 2: unconnected-(J11-Pin_2-Pad2) -> RTS
- J11 pad 6: unconnected-(J11-Pin_6-Pad6) -> DSR
- RN1 pad 8: SHIFT-CLOCK-VIA -> SHIFT-CLOCK
- U1 pad 12: /A4 -> /A0
- U1 pad 13: /A5 -> /A1
- U1 pad 14: /A6 -> /A2
- U1 pad 16: /A7 -> /A3
- U1 pad 18: /A8 -> /A4
- U1 pad 19: /B0 -> /A5
- U1 pad 20: /B1 -> /A6
- U1 pad 21: /B2 -> /A7
- U1 pad 22: /B3 -> /A8
- U1 pad 39: ~{RES} -> EMU
- U1 pad 40: SHIFT-CLOCK-VIA-3V3 -> SHIFT-CLOCK
- U1 pad 41: SHIFT-CLOCK-PIC-3V3 -> SHIFT-DATA
- U1 pad 42: SHIFT-DATA-3V3 -> ~{BOOT}
- U1 pad 5: /A0 -> /B0
- U1 pad 6: /A1 -> /B1
- U1 pad 7: /A2 -> /B2
- U1 pad 8: /A3 -> /B3
- U10 pad 11: /B7 -> /B0
- U10 pad 12: /B6 -> /B1
- U10 pad 13: /B5 -> /B2
- U10 pad 14: /B4 -> /B3
- U10 pad 15: /B3 -> /B4
- U10 pad 16: /B2 -> /B5
- U10 pad 17: /B1 -> /B6
- U10 pad 18: /B0 -> /B7
- U10 pad 2: /D0 -> /D7
- U10 pad 3: /D1 -> /D6
- U10 pad 4: /D2 -> /D5
- U10 pad 5: /D3 -> /D4
- U10 pad 6: /D4 -> /D3
- U10 pad 7: /D5 -> /D2
- U10 pad 8: /D6 -> /D1
- U10 pad 9: /D7 -> /D0
- U14 pad 1: +3.3V -> GND
- U14 pad 2: PHI2-3V3 -> ~{VIA-3V3}
- U14 pad 3: ~{VIA-3V3} -> GND
- U14 pad 4: SHIFT-CLOCK-VIA-3V3 -> ~{VIA}
- U14 pad 5: SHIFT-DATA-3V3 -> +5V
- U15 pad 11: /C7 -> /C0
- U15 pad 12: /C6 -> /C1
- U15 pad 13: /C5 -> /C2
- U15 pad 14: /C4 -> /C3
- U15 pad 15: /C3 -> /C4
- U15 pad 16: /C2 -> /C5
- U15 pad 17: /C1 -> /C6
- U15 pad 18: /C0 -> /C7
- U15 pad 2: /A0 -> /A7
- U15 pad 3: /A1 -> /A6
- U15 pad 4: /A2 -> /A5
- U15 pad 5: /A3 -> /A4
- U15 pad 6: /A4 -> /A3
- U15 pad 7: /A5 -> /A2
- U15 pad 8: /A6 -> /A1
- U15 pad 9: /A7 -> /A0
- U16 pad 11: /C15 -> /C8
- U16 pad 12: /C14 -> /C9
- U16 pad 13: /C13 -> /C10
- U16 pad 14: /C12 -> /C11
- U16 pad 15: /C11 -> /C12
- U16 pad 16: /C10 -> /C13
- U16 pad 17: /C9 -> /C14
- U16 pad 18: /C8 -> /C15
- U16 pad 2: /A8 -> /A15
- U16 pad 3: /A9 -> /A14
- U16 pad 4: /A10 -> /A13
- U16 pad 5: /A11 -> /A12
- U16 pad 6: /A12 -> /A11
- U16 pad 7: /A13 -> /A10
- U16 pad 8: /A14 -> /A9
- U16 pad 9: /A15 -> /A8
- U21 pad 10: /D6 -> /E6
- U21 pad 11: SHIFT-CLOCK-PIC-3V3 -> SPI-CLK
- U21 pad 12: SHIFT-DATA-3V3 -> SPI-MOSI
- U21 pad 14: SPI-CLK -> SPI-MISO
- U21 pad 15: SPI-MISO -> DSR
- U21 pad 16: SPI-MOSI -> RTS
- U21 pad 2: /D0 -> /E0
- U21 pad 23: ~{RW} -> ~{BOOT}
- U21 pad 3: /D1 -> /E1
- U21 pad 4: /D2 -> /E2
- U21 pad 5: /D3 -> /E3
- U21 pad 6: /D4 -> /E4
- U21 pad 7: /D5 -> /E5
- U21 pad 9: /D7 -> /E7
- U4 pad 33: unconnected-(U4-E-Pad33) -> EMU
- U5 pad 1: JOY-BUTTON2-A -> /E5
- U5 pad 10: JOY-BUTTON2-B -> KEY-DATA
- U5 pad 11: JOY-SELECT -> MOUSE-DATA
- U5 pad 13: SHIFT-CLOCK-VIA -> SHIFT-CLOCK
- U5 pad 2: MOUSE-DATA -> /E6
- U5 pad 3: KEY-DATA -> /E7
- U5 pad 4: JOY-UP-B -> JOY-CLOCK
- U5 pad 40: JOY-UP-A -> /E0
- U5 pad 41: JOY-DOWN-A -> /E1
- U5 pad 42: JOY-LEFT-A -> /E2
- U5 pad 43: JOY-RIGHT-A -> /E3
- U5 pad 44: JOY-BUTTON1-A -> /E4
- U5 pad 6: JOY-DOWN-B -> JOY-LATCH
- U5 pad 7: JOY-LEFT-B -> JOY-SELECT
- U5 pad 8: JOY-RIGHT-B -> JOY-DATA-A
- U5 pad 9: JOY-BUTTON1-B -> JOY-DATA-B
Routing:
- net +5V: track 70.6 -> 83.4 mm
- net GND: track 31.4 -> 37.8 mm, vias 15 -> 19
- net +3.3V: track 41.9 -> 40.9 mm

Commit message: Add files via upload
Parts:
- removed C29: C_Small, Capacitor_THT:C_Disc_D3.0mm_W2.0mm_P2.50mm
- removed Q1, Q2: PN2222A, Package_TO_SOT_THT:TO-92_HandSolder
- removed R1, R2: R_US, Resistor_THT:R_Axial_DIN0207_L6.3mm_D2.5mm_P2.54mm_Vertical
- removed U13, U14: 74AHCT1G125, Package_TO_SOT_SMD:SOT-23-5_HandSoldering
- added U12: 74AHCT08, Package_SO:SOIC-14_3.9x8.7mm_P1.27mm, F.Cu at (103.6, 120.7)
- moved R14 16.5 mm to (102.2, 80.0), turned to 0 degrees
- moved C22 14.5 mm to (110.5, 81.9)
- moved R16 13.1 mm to (102.2, 83.8), turned to 0 degrees
- moved C27 10.2 mm to (92.7, 134.6), turned to 0 degrees
- moved C14 7.64 mm to (103.5, 127.0), turned to 0 degrees
- moved U1 1.43 mm to (113.7, 93.3)
- moved C13 1.43 mm to (117.5, 84.4)
- moved C21 1.43 mm to (122.6, 92.7)
- moved C5 1.43 mm to (104.8, 87.7)
Routing:
- net +5V: track 83.4 -> 79.6 mm
- net GND: track 37.8 -> 37.7 mm, vias 19 -> 18

Commit message: Add files via upload
Parts:
- turned U12 to 0 degrees
Connections:
- U12 pad 10: unconnected-(U12-Pad10) -> PHI2-3V3
- U12 pad 11: unconnected-(U12-Pad11) -> WHITE-PIX-B
- U12 pad 12: unconnected-(U12-Pad12) -> TEXT-PIX-B
- U12 pad 13: unconnected-(U12-Pad13) -> ~{PHI2-3V3}
- U12 pad 2: ~{PHI2-3V3} -> PHI2-3V3
- U12 pad 5: VIA-3V3 -> ~{VIA-3V3}
- U12 pad 8: unconnected-(U12-Pad8) -> WHITE-PIX-A
- U12 pad 9: unconnected-(U12-Pad9) -> TEXT-PIX-A
Routing:
- net GND: track 37.7 -> 35.8 mm, vias 18 -> 17
- net +5V: track 79.6 -> 81.4 mm, vias 0 -> 1

Commit message: Add files via upload
Parts:
- turned U12 to 180 degrees
Routing:
- net GND: track 35.8 -> 37.7 mm, vias 17 -> 18
- net +5V: track 81.4 -> 79.6 mm, vias 1 -> 0
Changed lines of the file:
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@@
   )
   (footprint "Package_SO:SOIC-14_3.9x8.7mm_P1.27mm" (layer "F.Cu")
-    (at 103.57 120.65)
+    (at 103.57 120.65 180)
     (descr "SOIC, 14 Pin (JEDEC MS-012AB, https://www.analog.com/media/en/package-pcb-resources/package/pkg_pdf/soic_narrow-r/r_14.pdf), generated with kicad-footprint-generator ipc_gullwing_generator.py")
     (tags "SOIC SO")
@@
         (effects (font (size 1 1) (thickness 0.15)))
     )
-    (fp_text user "74AHCT08" (at -4.51 0.635 90 unlocked) (layer "F.SilkS")
+    (fp_text user "74AHCT08" (at 4.51 -0.635 90 unlocked) (layer "F.SilkS")
         (effects (font (size 1 1) (thickness 0.15)))
     )
@@
     (fp_line (start 1.95 4.325) (end -1.95 4.325)
       (stroke (width 0.1) (type solid)) (layer "F.Fab"))
-    (pad "1" smd roundrect (at -2.475 -3.81) (size 1.95 0.6) (layers "F.Cu" "F.Paste" "F.Mask") (roundrect_rratio 0.25)
+    (pad "1" smd roundrect (at -2.475 -3.81 180) (size 1.95 0.6) (layers "F.Cu" "F.Paste" "F.Mask") (roundrect_rratio 0.25)
       (net 1 "+5V") (pintype "input"))
-    (pad "2" smd roundrect (at -2.475 -2.54) (size 1.95 0.6) (layers "F.Cu" "F.Paste" "F.Mask") (roundrect_rratio 0.25)
+    (pad "2" smd roundrect (at -2.475 -2.54 180) (size 1.95 0.6) (layers "F.Cu" "F.Paste" "F.Mask") (roundrect_rratio 0.25)
       (net 57 "PHI2-3V3") (pintype "input"))
-    (pad "3" smd roundrect (at -2.475 -1.27) (size 1.95 0.6) (layers "F.Cu" "F.Paste" "F.Mask") (roundrect_rratio 0.25)
+    (pad "3" smd roundrect (at -2.475 -1.27 180) (size 1.95 0.6) (layers "F.Cu" "F.Paste" "F.Mask") (roundrect_rratio 0.25)
       (net 129 "PHI2") (pintype "output"))
-    (pad "4" smd roundrect (at -2.475 0) (size 1.95 0.6) (layers "F.Cu" "F.Paste" "F.Mask") (roundrect_rratio 0.25)
+    (pad "4" smd roundrect (at -2.475 0 180) (size 1.95 0.6) (layers "F.Cu" "F.Paste" "F.Mask") (roundrect_rratio 0.25)
       (net 1 "+5V") (pintype "input"))
-    (pad "5" smd roundrect (at -2.475 1.27) (size 1.95 0.6) (layers "F.Cu" "F.Paste" "F.Mask") (roundrect_rratio 0.25)
+    (pad "5" smd roundrect (at -2.475 1.27 180) (size 1.95 0.6) (layers "F.Cu" "F.Paste" "F.Mask") (roundrect_rratio 0.25)
       (net 174 "~{VIA-3V3}") (pintype "input"))
-    (pad "6" smd roundrect (at -2.475 2.54) (size 1.95 0.6) (layers "F.Cu" "F.Paste" "F.Mask") (roundrect_rratio 0.25)
+    (pad "6" smd roundrect (at -2.475 2.54 180) (size 1.95 0.6) (layers "F.Cu" "F.Paste" "F.Mask") (roundrect_rratio 0.25)
       (net 131 "~{VIA}") (pintype "output"))
-    (pad "7" smd roundrect (at -2.475 3.81) (size 1.95 0.6) (layers "F.Cu" "F.Paste" "F.Mask") (roundrect_rratio 0.25)
+    (pad "7" smd roundrect (at -2.475 3.81 180) (size 1.95 0.6) (layers "F.Cu" "F.Paste" "F.Mask") (roundrect_rratio 0.25)
       (net 2 "GND") (pinfunction "GND") (pintype "power_in"))
-    (pad "8" smd roundrect (at 2.475 3.81) (size 1.95 0.6) (layers "F.Cu" "F.Paste" "F.Mask") (roundrect_rratio 0.25)
+    (pad "8" smd roundrect (at 2.475 3.81 180) (size 1.95 0.6) (layers "F.Cu" "F.Paste" "F.Mask") (roundrect_rratio 0.25)
       (net 51 "WHITE-PIX-A") (pintype "output"))
-    (pad "9" smd roundrect (at 2.475 2.54) (size 1.95 0.6) (layers "F.Cu" "F.Paste" "F.Mask") (roundrect_rratio 0.25)
+    (pad "9" smd roundrect (at 2.475 2.54 180) (size 1.95 0.6) (layers "F.Cu" "F.Paste" "F.Mask") (roundrect_rratio 0.25)
       (net 52 "TEXT-PIX-A") (pintype "input"))
-    (pad "10" smd roundrect (at 2.475 1.27) (size 1.95 0.6) (layers "F.Cu" "F.Paste" "F.Mask") (roundrect_rratio 0.25)
+    (pad "10" smd roundrect (at 2.475 1.27 180) (size 1.95 0.6) (layers "F.Cu" "F.Paste" "F.Mask") (roundrect_rratio 0.25)
       (net 57 "PHI2-3V3") (pintype "input"))
-    (pad "11" smd roundrect (at 2.475 0) (size 1.95 0.6) (layers "F.Cu" "F.Paste" "F.Mask") (roundrect_rratio 0.25)
+    (pad "11" smd roundrect (at 2.475 0 180) (size 1.95 0.6) (layers "F.Cu" "F.Paste" "F.Mask") (roundrect_rratio 0.25)
       (net 53 "WHITE-PIX-B") (pintype "output"))
-    (pad "12" smd roundrect (at 2.475 -1.27) (size 1.95 0.6) (layers "F.Cu" "F.Paste" "F.Mask") (roundrect_rratio 0.25)
+    (pad "12" smd roundrect (at 2.475 -1.27 180) (size 1.95 0.6) (layers "F.Cu" "F.Paste" "F.Mask") (roundrect_rratio 0.25)
       (net 54 "TEXT-PIX-B") (pintype "input"))
-    (pad "13" smd roundrect (at 2.475 -2.54) (size 1.95 0.6) (layers "F.Cu" "F.Paste" "F.Mask") (roundrect_rratio 0.25)
+    (pad "13" smd roundrect (at 2.475 -2.54 180) (size 1.95 0.6) (layers "F.Cu" "F.Paste" "F.Mask") (roundrect_rratio 0.25)
       (net 58 "~{PHI2-3V3}") (pintype "input"))
-    (pad "14" smd roundrect (at 2.475 -3.81) (size 1.95 0.6) (layers "F.Cu" "F.Paste" "F.Mask") (roundrect_rratio 0.25)
+    (pad "14" smd roundrect (at 2.475 -3.81 180) (size 1.95 0.6) (layers "F.Cu" "F.Paste" "F.Mask") (roundrect_rratio 0.25)
       (net 1 "+5V") (pinfunction "VCC") (pintype "power_in"))
     (model "${KICAD6_3DMODEL_DIR}/Package_SO.3dshapes/SOIC-14_3.9x8.7mm_P1.27mm.wrl"
@@
   (segment (start 111.265 149.21) (end 111.265 152.3) (width 0.508) (layer "F.Cu") (net 1))
   (segment (start 137.795 153.275) (end 135.255 153.275) (width 0.508) (layer "F.Cu") (net 1))
-  (segment (start 106.045 116.84) (end 104.205 116.84) (width 0.508) (layer "F.Cu") (net 1))
   (segment (start 111.165 127) (end 111.165 131.445) (width 0.508) (layer "F.Cu") (net 1))
   (segment (start 71.755 121.92) (end 74.95 121.92) (width 0.508) (layer "F.Cu") (net 1))
@@
   (segment (start 127 104.775) (end 127 102.235) (width 0.508) (layer "F.Cu") (net 1))
   (segment (start 92.71 111.365) (end 95.25 111.365) (width 0.508) (layer "F.Cu") (net 1))
-  (via (at 104.205 116.84) (size 0.8) (drill 0.4) (layers "F.Cu" "B.Cu") (net 1))
   (segment (start 117.475 143.129) (end 117.894 142.71) (width 0.508) (layer "F.Cu") (net 2))
   (segment (start 152.02 100.965) (end 150.495 100.965) (width 0.508) (layer "F.Cu") (net 2))
@@
   (segment (start 123.825 145.175) (end 123.825 146.925) (width 0.508) (layer "F.Cu") (net 2))
   (segment (start 116.065 89.375) (end 116.065 87.645) (width 0.508) (layer "F.Cu") (net 2))
+  (segment (start 106.045 116.84) (end 104.205 116.84) (width 0.508) (layer "F.Cu") (net 2))
   (segment (start 117.856 143.51) (end 119.365 143.51) (width 0.508) (layer "F.Cu") (net 2))
   (segment (start 117.495 93.345) (end 119.365 93.345) (width 0.508) (layer "F.Cu") (net 2))
@@
   (via (at 67.775 80.18) (size 0.8) (drill 0.4) (layers "F.Cu" "B.Cu") (net 2))
   (via (at 117.475 143.129) (size 0.8) (drill 0.4) (layers "F.Cu" "B.Cu") (net 2))
+  (via (at 104.205 116.84) (size 0.8) (drill 0.4) (layers "F.Cu" "B.Cu") (net 2))
   (via (at 133.35 126.365) (size 0.8) (drill 0.4) (layers "F.Cu" "B.Cu") (net 2))
   (via (at 133.35 90.805) (size 0.8) (drill 0.4) (layers "F.Cu" "B.Cu") (net 2))
@@
     )
   )
+  (group "" (id 23c33717-44c8-44e4-869e-f67908dbf0d1)
+    (members
+      02fdd237-94cf-4eeb-bfa9-ab855244a659
+      1bfe771c-de59-4802-ac1f-5bfe987c95c5
+      6c576b43-8160-4a72-bcb2-5ccc907c7545
+      6fbddc10-24b8-482b-9395-9df413870231
+      7b8bfaf1-8b7c-4401-9cd0-3c7fa825d7f4
+      a284555b-34f8-49ce-88a8-3128ece8b229
+      a5b50d78-a37b-4e9e-a5c7-f50ed3021f4c
+      afd4bacc-ac44-464f-9f35-001d38f8b7d5
+      df1c0b5e-bf36-4a59-ba09-69c21e3946a5
+    )
+  )
