File: LastAcolyte6.kicad_pcb (KiCad board)
At the start: 4 copper layers, 100 x 100 mm, 87 parts, among them J1 Conn_02x23_Odd_Even, J10 DualPower_USB_B, J11 Conn_01x06, J2 DE9_Plug, J3 Conn_02x05_Odd_Even, J4 DE9_Plug, J5 DE15_Receptacle_HighDensity, J6 AudioJack3, J7 Mini-DIN-6, J8 Mini-DIN-6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

Commit message: Add files via upload
Parts:
- J1: footprint Connector_PinHeader_2.54mm:PinHeader_2x23_P2.54mm_Horizontal -> Connector_PinHeader_2.54mm:PinHeader_2x23_P2.54mm_Vertical
- moved G1001 1.30 mm to (117.5, 114.1)
- moved G1000 0.41 mm to (109.5, 107.0)
Routing:
- net ~{NMI}: track 0.00 -> 167.3 mm, vias 0 -> 3
- net /A6: track 0.00 -> 167.0 mm, vias 0 -> 5
- net /A7: track 0.00 -> 158.1 mm, vias 0 -> 7
- net ~{RES}: track 0.00 -> 156.3 mm, vias 0 -> 3
- net RDY: track 0.00 -> 156.0 mm, vias 0 -> 2
- net /A5: track 0.00 -> 150.2 mm, vias 0 -> 7
- net /A4: track 0.00 -> 146.5 mm, vias 0 -> 6
- net /A0: track 0.00 -> 146.3 mm, vias 0 -> 5
- net DSR: track 0.00 -> 144.6 mm
- net PHI2-3V3: track 0.00 -> 143.8 mm, vias 0 -> 6
- net TX/CK: track 0.00 -> 141.6 mm
- net /B3: track 0.00 -> 141.5 mm, vias 0 -> 2
- net /A2: track 0.00 -> 141.0 mm, vias 0 -> 6
- net ~{WR}: track 0.00 -> 138.1 mm, vias 0 -> 3
- net /A17: track 0.00 -> 137.1 mm, vias 0 -> 4
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Other:
- board text added: "+5V /WR /RD RDY"
- board text added: "+5V A0 A1 A2 A3"
- board text added: "/MCL /NMI /RES PHI2"
- board text added: "/ZERO"
- board text added: "A12 A13 A14 A15"
- board text added: "A4 A5 A6 A7 +5V"
- board text added: "B3 B4 B5 B6 B7"
- board text added: "D3 D2 D1 D0"
- board text added: "GND A16 A17 A18"
- board text added: "GND A8 A9 A10 A11"
- board text added: "GND D7 D6 D5 D4"
