File: LastAcolyte6.kicad_pcb (KiCad board)
At the start: 4 copper layers, 100 x 100 mm, 87 parts, among them J1 Conn_02x23_Odd_Even, J10 DualPower_USB_B, J11 Conn_01x06, J2 DE9_Plug, J3 Conn_02x05_Odd_Even, J4 DE9_Plug, J5 DE15_Receptacle_HighDensity, J6 AudioJack3, J7 Mini-DIN-6, J8 Mini-DIN-6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

Commit message: Add files via upload
Parts:
- added G102: LOGO, Library:Mystery, B.Cu at (146.8, 129.3)
Other:
- board text added: "Garth Wilson's 6502 Primer wilsonminesco.com Join the Forum 6502.org"
- board text added: "John 3:16 - For God so loved the world, that He gave His only begotten Son [Jesus], that whosoever believeth in Him should not perish, but have everlasting life."
- board text added: "Professor Steven Chad Burrow stevenchadburrow@gmail.com github.com/stevenchadburrow youtube.com/user/stevenchadburrow"
Changed lines of the file:
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@@
     )
   )
+  (footprint "Library:Mystery" (layer "B.Cu")
+    (at 146.812 129.286 -90)
+    (attr board_only exclude_from_pos_files exclude_from_bom)
+    (fp_text reference "G102" (at 0 0 -270) (layer "B.SilkS") hide
+        (effects (font (size 1.524 1.524) (thickness 0.3)) (justify mirror))
+    )
+    (fp_text value "LOGO" (at 0.75 0 -270) (layer "B.SilkS") hide
+        (effects (font (size 1.524 1.524) (thickness 0.3)) (justify mirror))
+    )
+    (fp_poly
+      (pts
+        (xy -1.75 1.501478)
+        (xy -1.25 1.501478)
+        (xy -1.25 1.000986)
+        (xy 1.25 1.000986)
+        (xy 1.25 1.501478)
+        (xy 1.75 1.501478)
+        (xy 1.75 2.001971)
+        (xy 3.75 2.001971)
+        (xy 3.75 1.501478)
+        (xy 2.25 1.501478)
+        (xy 2.25 1.000986)
+        (xy 1.75 1.000986)
+        (xy 1.75 0.500493)
+        (xy 3.25 0.500493)
+        (xy 3.25 0)
+        (xy 3.75 0)
+        (xy 3.75 -1.000985)
+        (xy 3.25 -1.000985)
+        (xy 3.25 -1.501477)
+        (xy 1.75 -1.501477)
+        (xy 1.75 -2.00197)
+        (xy -1.75 -2.00197)
+        (xy -1.75 -1.501477)
+        (xy -3.25 -1.501477)
+        (xy -3.25 -1.000985)
+        (xy -3.75 -1.000985)
+        (xy -3.75 -0.500492)
+        (xy -1.75 -0.500492)
+        (xy -1.25 -0.500492)
+        (xy 1.25 -0.500492)
+        (xy 1.75 -0.500492)
+        (xy 1.75 0)
+        (xy 1.25 0)
+        (xy 1.25 -0.500492)
+        (xy -1.25 -0.500492)
+        (xy -1.25 0)
+        (xy -1.75 0)
+        (xy -1.75 -0.500492)
+        (xy -3.75 -0.500492)
+        (xy -3.75 0)
+        (xy -3.25 0)
+        (xy -3.25 0.500493)
+        (xy -1.75 0.500493)
+        (xy -1.75 1.000986)
+        (xy -2.25 1.000986)
+        (xy -2.25 1.501478)
+        (xy -3.75 1.501478)
+        (xy -3.75 2.001971)
+        (xy -1.75 2.001971)
+      )
+      (stroke (width 0) (type solid)) (fill solid) (layer "B.SilkS"))
+  )
   (gr_line (start 108.015 123.825) (end 108.015 125.095)
     (stroke (width 0.15) (type default)) (layer "F.SilkS"))
@@
   (gr_line (start 63.5 63.5) (end 63.5 163.5)
     (stroke (width 0.1) (type default)) (layer "Edge.Cuts"))
+  (gr_text "John 3:16 - For God so loved the world, \n  that He gave His only begotten Son [Jesus], \n  that whosoever believeth in Him should not perish, \n  but have everlasting life." (at 134.62 90.17 90) (layer "B.SilkS")
+    (effects (font (size 1 1) (thickness 0.15)) (justify left mirror))
+  )
+  (gr_text "Professor Steven Chad Burrow\nstevenchadburrow@gmail.com\ngithub.com/stevenchadburrow\nyoutube.com/user/stevenchadburrow" (at 147.066 90.17 90) (layer "B.SilkS")
+    (effects (font (size 1.5 1.5) (thickness 0.225)) (justify left mirror))
+  )
+  (gr_text "Garth Wilson's\n6502 Primer \nwilsonminesco.com\nJoin the Forum\n6502.org" (at 147.32 149.86 90) (layer "B.SilkS")
+    (effects (font (size 1.25 1.25) (thickness 0.175)) (justify mirror))
+  )
   (gr_text "+" (at 109.641 130.81 180) (layer "F.SilkS")
     (effects (font (size 1 1) (thickness 0.15)) (justify bottom))

Commit message: Add files via upload
Parts:
- turned C14 to 180 degrees
Routing:
- net PHI2-3V3: track 143.8 -> 148.7 mm
- net +5V: track 119.1 -> 115.9 mm, vias 4 -> 5
