File: LastAcolyte6.kicad_sch (KiCad schematic)
At the start: 83 parts, among them J1 Conn_02x23_Odd_Even, J1 DE9_Plug, J10 DualPower_USB_B, J11 Conn_01x06, J11 Micro_SD_Card, J3 DE15_Receptacle_HighDensity, J5 Mini-DIN-6, J6 AudioJack3, J7 Mini-DIN-6, J8 DE9_Plug, J9 Conn_02x05_Odd_Even, Q1 PN2222A, Q2 PN2222A, SW1 SW_Push, SW1 SW_SPDT, U1 XC9572VQ44, U10 74AHCT245, U14 TXB0104D, U15 74AHCT245, U16 74AHCT245, U19 74AHCT374, U2 IS61C5128AL-10KLI, U21 PIC16F886-IP, U4 W65C816SxQ, U5 W65C22SxQ, U6 74AHCT273, U7 IS61C5128AL-10KLI, U8 LM1117MP-3.3, X1 CXO_DIP8

Commit message: Add files via upload
Connections:
- net A0: now also J1.18 (Pin_18); no longer J1.36 (Pin_36)
- net A1: now also J1.16 (Pin_16); no longer J1.34 (Pin_34)
- net A16: now also J1.7 (Pin_7); no longer J1.18 (Pin_18)
- net A17: now also J1.5 (Pin_5); no longer J1.16 (Pin_16)
- net A18: now also J1.3 (Pin_3); no longer J1.14 (Pin_14)
- net A2: now also J1.14 (Pin_14); no longer J1.32 (Pin_32)
- net A3: now also J1.12 (Pin_12); no longer J1.30 (Pin_30)
- net A4: now also J1.10 (Pin_10); no longer J1.28 (Pin_28)
- net A5: now also J1.8 (Pin_8); no longer J1.26 (Pin_26)
- net A6: now also J1.6 (Pin_6); no longer J1.24 (Pin_24)
- net A7: now also J1.4 (Pin_4); no longer J1.22 (Pin_22)
- net B3: now also J1.30 (Pin_30); no longer J1.12 (Pin_12)
- net B4: now also J1.28 (Pin_28); no longer J1.10 (Pin_10)
- net B5: now also J1.26 (Pin_26); no longer J1.8 (Pin_8)
- net B6: now also J1.24 (Pin_24); no longer J1.6 (Pin_6)
- net B7: now also J1.22 (Pin_22); no longer J1.4 (Pin_4)
- net PHI2: now also J1.40 (Pin_40); no longer J1.1 (Pin_1)
- net RDY: now also J1.32 (Pin_32); no longer J1.40 (Pin_40)
- net ~{RD}: now also J1.34 (Pin_34); no longer J1.5 (Pin_5)
- net ~{WR}: now also J1.36 (Pin_36); no longer J1.7 (Pin_7)
- net ~{ZERO}: now also J1.1 (Pin_1); no longer J1.3 (Pin_3)

Commit message: Add files via upload
Parts:
- removed C20: C_Small, Capacitor_THT:C_Disc_D3.0mm_W2.0mm_P2.50mm, symbol Device:C_Small
- removed U14: TXB0104D, Package_SO:SOIC-14_3.9x8.7mm_P1.27mm, symbol Logic_LevelTranslator:TXB0104D
- added C12, C23 (x3): C_Small, Capacitor_THT:C_Disc_D3.0mm_W2.0mm_P2.50mm, symbol Device:C_Small
- added R10: R_US, Resistor_THT:R_Axial_DIN0207_L6.3mm_D2.5mm_P2.54mm_Vertical, symbol Device:R_US
- added U11: 74AHCT245, LastAcolyte6:SOIC-20-Adj_7.5x12.8mm_P1.27mm, symbol 74xx:74HC245
- added U13, U14: 74AHCT1G125, Package_TO_SOT_SMD:SOT-23-5_HandSoldering, symbol 74xGxx:74LVC1G125
- added U8, U9: 74HCT166, Package_SO:SOIC-16_3.9x9.9mm_P1.27mm, symbol 74xx:74LS166
- J11: Field4 FT232RL 3.3V -> FT232RL
Connections:
- net SHIFT-CLOCK-VIA-3V3 is gone; now on net SHIFT-CLOCK: U1.40 (P2)
- net +5V: now also C12.2, C23.2, C23.2, C23.2, U11.20 (VCC), U13.5 (VCC), U14.5 (VCC), U8.1 (Ds), U8.16 (VCC), U8.2 (A), U8.3 (B), U8.9 (Clr), U9.1 (Ds), U9.16 (VCC), U9.2 (A), U9.3 (B), U9.9 (Clr)
- net A0: now also U1.12 (P18), U15.9 (A7); no longer U1.5 (P11), U15.2 (A0)
- net A1: now also U1.13 (P19), U15.8 (A6); no longer U1.6 (P12), U15.3 (A1)
- net A10: now also U16.7 (A5); no longer U16.4 (A2)
- net A11: now also U16.6 (A4); no longer U16.5 (A3)
- net A12: now also U16.5 (A3); no longer U16.6 (A4)
- net A13: now also U16.4 (A2); no longer U16.7 (A5)
- net A14: now also U16.3 (A1); no longer U16.8 (A6)
- net A15: now also U16.2 (A0); no longer U16.9 (A7)
- net A2: now also U1.14 (P20), U15.7 (A5); no longer U1.7 (P13), U15.4 (A2)
- net A3: now also U1.16 (P22), U15.6 (A4); no longer U1.8 (P14), U15.5 (A3)
- net A4: now also U1.18 (P24), U15.5 (A3); no longer U1.12 (P18), U15.6 (A4)
- net A5: now also U1.19 (P25), U15.4 (A2); no longer U1.13 (P19), U15.7 (A5)
- net A6: now also U1.20 (P26), U15.3 (A1); no longer U1.14 (P20), U15.8 (A6)
- net A7: now also U1.21 (P27), U15.2 (A0); no longer U1.16 (P22), U15.9 (A7)
- net A8: now also U1.22 (P28), U16.9 (A7); no longer U1.18 (P24), U16.2 (A0)
- net A9: now also U16.8 (A6); no longer U16.3 (A1)
- net B0: now also U1.5 (P11), U10.11 (B7); no longer U1.19 (P25), U10.18 (B0)
- net B1: now also U1.6 (P12), U10.12 (B6); no longer U1.20 (P26), U10.17 (B1)
- net B2: now also U1.7 (P13), U10.13 (B5); no longer U1.21 (P27), U10.16 (B2)
- net B3: now also U1.8 (P14), U10.14 (B4); no longer U1.22 (P28), U10.15 (B3)
- net B4: now also U10.15 (B3); no longer U10.14 (B4)
- net B5: now also U10.16 (B2); no longer U10.13 (B5)
- net B6: now also U10.17 (B1); no longer U10.12 (B6)
- net B7: now also U10.18 (B0); no longer U10.11 (B7)
- net C0: now also U15.11 (B7); no longer U15.18 (B0)
- net C1: now also U15.12 (B6); no longer U15.17 (B1)
- net C10: now also U16.13 (B5); no longer U16.16 (B2)
- net C11: now also U16.14 (B4); no longer U16.15 (B3)
- net C12: now also U16.15 (B3); no longer U16.14 (B4)
- net C13: now also U16.16 (B2); no longer U16.13 (B5)
- net C14: now also U16.17 (B1); no longer U16.12 (B6)
- net C15: now also U16.18 (B0); no longer U16.11 (B7)
- net C2: now also U15.13 (B5); no longer U15.16 (B2)
- net C3: now also U15.14 (B4); no longer U15.15 (B3)
- net C4: now also U15.15 (B3); no longer U15.14 (B4)
- net C5: now also U15.16 (B2); no longer U15.13 (B5)
- net C6: now also U15.17 (B1); no longer U15.12 (B6)
- net C7: now also U15.18 (B0); no longer U15.11 (B7)
- net C8: now also U16.11 (B7); no longer U16.18 (B0)
- net C9: now also U16.12 (B6); no longer U16.17 (B1)
- net D0: now also U10.9 (A7), U11.18 (B0); no longer U10.2 (A0), U21.2 (ULPWU/C12IN0-/AN0/RA0)
- net D1: now also U10.8 (A6), U11.17 (B1); no longer U10.3 (A1), U21.3 (C12IN1-/AN1/RA1)
- net D2: now also U10.7 (A5), U11.16 (B2); no longer U10.4 (A2), U21.4 (CVref/C2IN1+/Vref-/AN2/RA2)
- net D3: now also U10.6 (A4), U11.15 (B3); no longer U10.5 (A3), U21.5 (C1IN+/Vref+/AN3/RA3)
- net D4: now also U10.5 (A3), U11.14 (B4); no longer U10.6 (A4), U21.6 (T0CKI/C1OUT/RA4)
- net D5: now also U10.4 (A2), U11.13 (B5); no longer U10.7 (A5), U21.7 (~{SS}/C2OUT/AN4/RA5)
- net D6: now also U10.3 (A1), U11.12 (B6); no longer U10.8 (A6), U21.10 (CLKOUT/OSC2/RA6)
- net D7: now also U10.2 (A0), U11.11 (B7); no longer U10.9 (A7), U21.9 (CLKIN/OSC1/RA7)
- net GND: now also C12.1, C23.1, C23.1, C23.1, R10.2, U11.10 (GND), U13.1, U13.3 (GND), U14.1, U14.3 (GND), U8.6 (CE), U8.8 (GND), U9.6 (CE), U9.8 (GND)
- net JOY-BUTTON1-A: now also U8.5 (D); no longer U5.44 (PA4)
- net JOY-BUTTON1-B: now also U9.5 (D); no longer U5.9 (PB4)
- net JOY-BUTTON2-A: now also U8.4 (C); no longer U5.1 (PA5)
- net JOY-BUTTON2-B: now also U9.4 (C); no longer U5.10 (PB5)
- net JOY-DOWN-A: now also U8.12 (G); no longer U5.41 (PA1)
- net JOY-DOWN-B: now also U9.12 (G); no longer U5.6 (PB1)
- net JOY-LEFT-A: now also U8.11 (F); no longer U5.42 (PA2)
- net JOY-LEFT-B: now also U9.11 (F); no longer U5.7 (PB2)
- net JOY-RIGHT-A: now also U8.10 (E); no longer U5.43 (PA3)
- net JOY-RIGHT-B: now also U9.10 (E); no longer U5.8 (PB3)
- net JOY-SELECT: now also U5.7 (PB2); no longer U5.11 (PB6)
- net JOY-UP-A: now also U8.14 (H); no longer U5.40 (PA0)
- net JOY-UP-B: now also U9.14 (H); no longer U5.4 (PB0)
- net KEY-DATA: now also U5.10 (PB5); no longer U5.3 (PA7)
- net MOUSE-DATA: now also U5.11 (PB6); no longer U5.2 (PA6)
- net PHI2: now also U13.4
- net PHI2-3V3: now also U13.2
- net SHIFT-DATA: now also U1.41 (P3)
- net SPI-CLK: now also U21.11 (RC0/T1OSO/T1CK1); no longer U21.14 (RC3/SCK/SCL)
- net SPI-MISO: now also U21.14 (RC3/SCK/SCL); no longer U21.15 (RC4/SDI/SDA)
- net SPI-MOSI: now also U21.12 (RC1/T1OSI/CCP2); no longer U21.16 (RC5/SDO)
- net ~{RES}: no longer U1.39 (P1)
- net ~{RW}: now also U11.1 (A->B); no longer U21.23 (P1B/AN8/RB2)
- net ~{VIA-3V3}: now also U14.2
- net ~{VIA}: now also U14.4
- net RTS: now reaches J11.2 (Pin_2)
- net RTS: now also U21.16 (RC5/SDO)
- net DSR: now reaches J11.6 (Pin_6)
- net DSR: now also U21.15 (RC4/SDI/SDA)
- net EMU: now reaches U4.33 (E)
- net EMU: now also U1.39 (P1)
- removed net SHIFT-CLOCK-PIC-3V3: U1.41 (P3), U21.11 (RC0/T1OSO/T1CK1)
- net SHIFT-CLOCK-VIA renamed SHIFT-CLOCK
- net SHIFT-DATA-3V3 renamed ~{BOOT}
- net ~{BOOT}: now also U21.23 (P1B/AN8/RB2), R10.1, U11.19 (CE); no longer U21.12 (RC1/T1OSI/CCP2)
- new net E0: U11.2 (A0), U21.2 (ULPWU/C12IN0-/AN0/RA0), U5.40 (PA0)
- new net E1: U11.3 (A1), U21.3 (C12IN1-/AN1/RA1), U5.41 (PA1)
- new net E2: U11.4 (A2), U21.4 (CVref/C2IN1+/Vref-/AN2/RA2), U5.42 (PA2)
- new net E3: U11.5 (A3), U21.5 (C1IN+/Vref+/AN3/RA3), U5.43 (PA3)
- new net E4: U11.6 (A4), U21.6 (T0CKI/C1OUT/RA4), U5.44 (PA4)
- new net E5: U11.7 (A5), U21.7 (~{SS}/C2OUT/AN4/RA5), U5.1 (PA5)
- new net E6: U11.8 (A6), U21.10 (CLKOUT/OSC2/RA6), U5.2 (PA6)
- new net E7: U11.9 (A7), U21.9 (CLKIN/OSC1/RA7), U5.3 (PA7)
- new net JOY-CLOCK: U5.4 (PB0), U8.7 (Clk), U9.7 (Clk)
- new net JOY-DATA-A: U5.8 (PB3), U8.13 (Qh)
- new net JOY-DATA-B: U5.9 (PB4), U9.13 (Qh)
- new net JOY-LATCH: U5.6 (PB1), U8.15 (PE), U9.15 (PE)
- no-connect marks 28 -> 25

Commit message: Add files via upload
Parts:
- removed C23: C_Small, Capacitor_THT:C_Disc_D3.0mm_W2.0mm_P2.50mm, symbol Device:C_Small
- removed Q1, Q2: PN2222A, Package_TO_SOT_THT:TO-92_HandSolder, symbol Transistor_BJT:PN2222A
- removed R1, R2: R_US, Resistor_THT:R_Axial_DIN0207_L6.3mm_D2.5mm_P2.54mm_Vertical, symbol Device:R_US
- removed U13, U14: 74AHCT1G125, Package_TO_SOT_SMD:SOT-23-5_HandSoldering, symbol 74xGxx:74LVC1G125
- added U12: 74AHCT08, symbol 74xx:74LS08
Connections:
- net +5V: now also U12.1, U12.14 (VCC), U12.4
- net GND: now also U12.7 (GND)
- net PHI2: now also U12.3
- net PHI2-3V3: now also U12.10, U12.2
- net TEXT-PIX-A: now also U12.9
- net TEXT-PIX-B: now also U12.12
- net WHITE-PIX-A: now also U12.8
- net WHITE-PIX-B: now also U12.11
- net ~{PHI2-3V3}: now also U12.13
- net ~{VIA-3V3}: now also U12.5
- net ~{VIA}: now also U12.6
Other:
- note removed: "Make sure these PN2222's will work here, or if we need something 'faster'? Or if they will work at all!"

Commit message: Add files via upload
Parts:
- U12: footprint (none) -> Package_SO:SOIC-14_3.9x8.7mm_P1.27mm
Changed lines of the file:
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@@
       (effects (font (size 1.27 1.27)))
     )
-    (property "Footprint" "" (at 355.6 214.63 0)
+    (property "Footprint" "Package_SO:SOIC-14_3.9x8.7mm_P1.27mm" (at 355.6 214.63 0)
       (effects (font (size 1.27 1.27)) hide)
     )
@@
       (effects (font (size 1.27 1.27)))
     )
-    (property "Footprint" "" (at 355.6 199.39 0)
+    (property "Footprint" "Package_SO:SOIC-14_3.9x8.7mm_P1.27mm" (at 355.6 199.39 0)
       (effects (font (size 1.27 1.27)) hide)
     )
@@
       (effects (font (size 1.27 1.27)))
     )
-    (property "Footprint" "" (at 355.6 229.87 0)
+    (property "Footprint" "Package_SO:SOIC-14_3.9x8.7mm_P1.27mm" (at 355.6 229.87 0)
       (effects (font (size 1.27 1.27)) hide)
     )
@@
       (effects (font (size 1.27 1.27)) (justify left))
     )
-    (property "Footprint" "" (at 387.35 219.71 0)
+    (property "Footprint" "Package_SO:SOIC-14_3.9x8.7mm_P1.27mm" (at 387.35 219.71 0)
       (effects (font (size 1.27 1.27)) hide)
     )
@@
       (effects (font (size 1.27 1.27)))
     )
-    (property "Footprint" "" (at 355.6 245.11 0)
+    (property "Footprint" "Package_SO:SOIC-14_3.9x8.7mm_P1.27mm" (at 355.6 245.11 0)
       (effects (font (size 1.27 1.27)) hide)
     )

Commit message: Add files via upload
Parts:
- J1: footprint Connector_PinHeader_2.54mm:PinHeader_2x23_P2.54mm_Horizontal -> Connector_PinHeader_2.54mm:PinHeader_2x23_P2.54mm_Vertical
Changed lines of the file:
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@@
       (effects (font (size 1.27 1.27)) hide)
     )
-    (property "Footprint" "Connector_PinHeader_2.54mm:PinHeader_2x23_P2.54mm_Horizontal" (at 541.02 215.9 0)
+    (property "Footprint" "Connector_PinHeader_2.54mm:PinHeader_2x23_P2.54mm_Vertical" (at 541.02 215.9 0)
       (effects (font (size 1.27 1.27)) hide)
     )
